File: input_buff.brd (EAGLE design)
At the start: 100.6 x 80.6 mm, 37 parts, among them X1 057-010-1, X2 057-016-1

Commit message: change led to cms, add addtionnal capa place
add an addtionnal 1206 capa before ldo
change led to 0805 smd
Parts:
- added C6: 10uF, resistor:C1210
- LED1: value (none) -> RED LED; device led:LED3MM -> led:CHIPLED_0805
- SL1: value (none) -> POW
- moved R4 8.89 mm to (26.7, 26.0)
- moved TP20 8.89 mm to (26.7, 23.5)
- moved TP17 4.62 mm to (29.2, 26.0)
- moved LED1 3.86 mm to (22.9, 26.0)
- moved TP18 2.01 mm to (10.2, 26.0)
- moved R5 0.63 mm to (31.8, 26.0)
- moved TP21 0.63 mm to (31.8, 23.5)
- turned R3 to 270 degrees
Connections:
- net GND: now also C6.2
- net N$3: now also LED1.C; no longer LED1.K
- net VIN: now also C6.1
Routing:
- net VIN: track 39.0 -> 43.5 mm
- net GND: track 12.4 -> 9.13 mm
- net N$3: track 6.48 -> 4.23 mm
- net 1V8: track 36.3 -> 37.4 mm
- net N$4: track 1.90 -> 2.85 mm

Commit message: final design + matching gerbers (production files)
Parts:
- removed SL1: POW, con-amp-quick:02P
- added R6: 4.7k, resistor:M0805
- added SL2: POW, con-amp-quick:02P
- added X3: 22-23-2021, con-molex:22-23-2021
Connections:
- new net !OE: R6.2, SL2.2, U$3.22
- net GND: now also R6.1, X3.1; no longer SL1.2, U$3.22
- net VIN: now also SL2.1, X3.2; no longer SL1.1
Routing:
- net VIN: track 43.5 -> 76.4 mm
- net !OE: track 0.00 -> 21.2 mm
- net GND: track 9.13 -> 7.75 mm
Changed lines of the file:
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@@
 <?xml version="1.0" encoding="utf-8"?>
 <!DOCTYPE eagle SYSTEM "eagle.dtd">
-<eagle version="6.1">
+<eagle version="6.0">
 <drawing>
 <settings>
@@
 <attribute name="OC_FARNELL" value="unknown" x="41.91" y="15.24" size="1.778" layer="27" rot="R270" display="off"/>
 </element>
-<element name="SL1" library="con-amp-quick" package="02P" value="POW" x="5.08" y="26.67" smashed="yes" rot="R90">
-<attribute name="OC_NEWARK" value="unknown" x="5.08" y="26.67" size="1.778" layer="27" rot="R90" display="off"/>
-<attribute name="MPN" value="" x="5.08" y="26.67" size="1.778" layer="27" rot="R90" display="off"/>
-<attribute name="MF" value="" x="5.08" y="26.67" size="1.778" layer="27" rot="R90" display="off"/>
-<attribute name="OC_FARNELL" value="unknown" x="5.08" y="26.67" size="1.778" layer="27" rot="R90" display="off"/>
-</element>
 <element name="TP17" library="testpad" package="TP10R" value="TPTP10R" x="29.21" y="26.035" smashed="yes">
 <attribute name="TP_SIGNAL_NAME" value="" x="29.21" y="24.13" size="1" layer="37"/>
@@
 <element name="LED1" library="led" package="CHIPLED_0805" value="RED LED" x="22.86" y="26.035" smashed="yes" rot="R180">
 <attribute name="NAME" x="20.955" y="30.48" size="0.8128" layer="25" font="fixed" rot="R270"/>
+</element>
+<element name="R6" library="resistor" package="M0805" value="4.7k" x="31.75" y="20.32" smashed="yes" rot="R270">
+<attribute name="NAME" x="33.401" y="23.876" size="1.27" layer="25" rot="R270"/>
+</element>
+<element name="SL2" library="con-amp-quick" package="02P" value="POW" x="35.56" y="26.67" smashed="yes" rot="R270">
+<attribute name="OC_NEWARK" value="unknown" x="35.56" y="26.67" size="1.778" layer="27" rot="R270" display="off"/>
+<attribute name="MPN" value="" x="35.56" y="26.67" size="1.778" layer="27" rot="R270" display="off"/>
+<attribute name="MF" value="" x="35.56" y="26.67" size="1.778" layer="27" rot="R270" display="off"/>
+<attribute name="OC_FARNELL" value="unknown" x="35.56" y="26.67" size="1.778" layer="27" rot="R270" display="off"/>
+</element>
+<element name="X3" library="con-molex" package="22-23-2021" value="22-23-2021" x="5.08" y="26.67" smashed="yes" rot="R270">
+<attribute name="OC_NEWARK" value="25C3832" x="5.08" y="26.67" size="1.778" layer="27" rot="R270" display="off"/>
+<attribute name="MPN" value="22-23-2021" x="5.08" y="26.67" size="1.778" layer="27" rot="R270" display="off"/>
+<attribute name="MF" value="MOLEX" x="5.08" y="26.67" size="1.778" layer="27" rot="R270" display="off"/>
+<attribute name="OC_FARNELL" value="1462926" x="5.08" y="26.67" size="1.778" layer="27" rot="R270" display="off"/>
 </element>
 </elements>
@@
 <contactref element="U$3" pad="1"/>
 <contactref element="C4" pad="1"/>
-<contactref element="SL1" pad="1"/>
 <contactref element="TP18" pad="TP"/>
 <contactref element="R1" pad="2"/>
@@
 <wire x1="14.605" y1="21.27" x2="15.56" y2="21.27" width="0.6096" layer="1"/>
 <wire x1="15.56" y1="21.27" x2="17.145" y2="19.685" width="0.6096" layer="1"/>
-<wire x1="5.08" y1="25.4" x2="10.16" y2="25.4" width="0.6096" layer="1"/>
 <wire x1="10.16" y1="25.4" x2="12.065" y2="25.4" width="0.6096" layer="1"/>
 <wire x1="14.605" y1="22.86" x2="14.605" y2="24.635" width="0.6096" layer="1"/>
@@
 <wire x1="14.605" y1="22.86" x2="14.605" y2="24.635" width="0.4064" layer="1"/>
 <wire x1="14.605" y1="21.27" x2="14.605" y2="22.225" width="0.4064" layer="1"/>
+<contactref element="SL2" pad="1"/>
+<wire x1="35.56" y1="27.94" x2="18.415" y2="27.94" width="0.4064" layer="16"/>
+<wire x1="18.415" y1="27.94" x2="12.7" y2="27.94" width="0.4064" layer="16"/>
+<wire x1="12.7" y1="27.94" x2="11.1125" y2="26.3525" width="0.4064" layer="16"/>
+<contactref element="X3" pad="2"/>
+<wire x1="11.1125" y1="26.3525" x2="10.16" y2="25.4" width="0.4064" layer="16"/>
+<wire x1="5.08" y1="25.4" x2="10.16" y2="25.4" width="0.4064" layer="16"/>
+<wire x1="10.16" y1="25.4" x2="11.1125" y2="26.3525" width="0.4064" layer="16"/>
+<wire x1="10.16" y1="25.4" x2="5.08" y2="25.4" width="0.6096" layer="1"/>
 </signal>
 <signal name="N$2">
@@
 <contactref element="C5" pad="1"/>
 <contactref element="TP17" pad="TP"/>
-<wire x1="26.435" y1="12.465" x2="26.67" y2="12.7" width="0.4064" layer="1"/>
+<wire x1="26.435" y1="12.465" x2="26.67" y2="12.7" width="0.6096" layer="1"/>
 <wire x1="25.785" y1="11.815" x2="26.435" y2="12.465" width="0.6096" layer="1"/>
 <wire x1="23.81" y1="19.12" x2="26.32" y2="19.12" width="0.6096" layer="1"/>
 <wire x1="26.32" y1="19.12" x2="26.67" y2="19.47" width="0.4064" layer="1"/>
 <wire x1="26.67" y1="19.47" x2="26.67" y2="19.685" width="0.4064" layer="1"/>
-<wire x1="25.785" y1="11.815" x2="25.785" y2="11.2022" width="0.4064" layer="1"/>
+<wire x1="25.785" y1="11.815" x2="25.785" y2="11.2022" width="0.6096" layer="1"/>
 <wire x1="25.785" y1="11.2022" x2="25.7778" y2="11.195" width="0.4064" layer="1"/>
 <wire x1="25.7778" y1="11.195" x2="25.7778" y2="10.545" width="0.3048" layer="1"/>
@@
 <contactref element="C2" pad="2"/>
 <contactref element="C4" pad="2"/>
-<contactref element="U$3" pad="22"/>
 <contactref element="X2" pad="2"/>
 <contactref element="X2" pad="16"/>
@@
 <wire x1="6.35" y1="6.35" x2="3.81" y2="6.35" width="0.4064" layer="1"/>
 <wire x1="26.67" y1="16.09" x2="26.455" y2="15.875" width="0.4064" layer="1"/>
-<wire x1="25.7778" y1="9.895" x2="24.395" y2="9.895" width="0.3048" layer="1"/>
 <polygon width="0.4064" layer="16" isolate="0.3048">
 <vertex x="-0.635" y="-0.635"/>
@@
 </polygon>
 <contactref element="TP19" pad="TP"/>
-<contactref element="SL1" pad="2"/>
 <contactref element="C6" pad="2"/>
+<contactref element="R6" pad="1"/>
+<contactref element="X3" pad="1"/>
 </signal>
 <signal name="OUT_0">
@@
 <wire x1="31.75" y1="25.085" x2="31.75" y2="25.4" width="0.4064" layer="1"/>
 </signal>
+<signal name="!OE">
+<contactref element="U$3" pad="22"/>
+<contactref element="R6" pad="2"/>
+<wire x1="25.7778" y1="9.895" x2="26.67" y2="9.895" width="0.3048" layer="1"/>
+<wire x1="26.67" y1="9.895" x2="26.67" y2="10.16" width="0.3048" layer="1"/>
+<wire x1="26.67" y1="10.16" x2="26.67" y2="11.43" width="0.3048" layer="1"/>
+<wire x1="26.67" y1="11.43" x2="29.21" y2="13.97" width="0.4064" layer="1"/>
+<wire x1="29.21" y1="13.97" x2="29.21" y2="17.145" width="0.4064" layer="1"/>
+<wire x1="29.21" y1="17.145" x2="29.21" y2="17.78" width="0.4064" layer="1"/>
+<wire x1="29.21" y1="17.78" x2="31.115" y2="19.685" width="0.4064" layer="1"/>
+<wire x1="31.115" y1="19.685" x2="31.435" y2="19.685" width="0.4064" layer="1"/>
+<wire x1="31.435" y1="19.685" x2="31.75" y2="19.37" width="0.4064" layer="1"/>
+<contactref element="SL2" pad="2"/>
+<wire x1="35.56" y1="25.4" x2="35.56" y2="22.86" width="0.4064" layer="1"/>
+<wire x1="35.56" y1="22.86" x2="31.75" y2="19.05" width="0.4064" layer="1"/>
+<wire x1="31.75" y1="19.37" x2="31.75" y2="19.05" width="0" layer="19" extent="1-1"/>
+</signal>
 </signals>
